File: ledpower.kicad_sch (KiCad schematic)
At the start: 2 parts

Commit message: V0.1
really jjust updating a bunch of stuff
Parts:
- removed U?: NCP1117ST20T3G, Package_TO_SOT_SMD:SOT-223-3_TabPin2, symbol Regulator_Linear:NCP1117-1.5_SOT223
- added C?: 10uF, symbol Device:C_Polarized
Connections:
- net GND: now also C?.2
- net 2V: now reaches J?.1
- net 2V: now also C?.1
Other:
- moved on the sheet: J?
Changed lines of the file:
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@@
 (kicad_sch (version 20230121) (generator eeschema)
   (paper "A4")
-  (junction (at 130.81 95.885) (diameter 0) (color 0 0 0 0)
+  (junction (at 131.445 97.155) (diameter 0) (color 0 0 0 0)
   )
-  (wire (pts (xy 102.87 86.995) (xy 123.19 86.995))
+  (wire (pts (xy 118.11 97.155) (xy 131.445 97.155))
     (stroke (width 0) (type default))
   )
-  (wire (pts (xy 130.81 94.615) (xy 130.81 95.885))
+  (wire (pts (xy 131.445 107.315) (xy 131.445 108.585))
     (stroke (width 0) (type default))
   )
-  (wire (pts (xy 115.57 92.075) (xy 115.57 95.885))
+  (wire (pts (xy 118.11 102.235) (xy 119.38 102.235))
     (stroke (width 0) (type default))
   )
-  (wire (pts (xy 115.57 95.885) (xy 130.81 95.885))
+  (wire (pts (xy 131.445 97.155) (xy 131.445 99.695))
     (stroke (width 0) (type default))
   )
-  (wire (pts (xy 115.57 92.075) (xy 102.87 92.075))
+  (wire (pts (xy 119.38 102.235) (xy 119.38 108.585))
     (stroke (width 0) (type default))
   )
-  (wire (pts (xy 130.81 95.885) (xy 130.81 98.425))
+  (wire (pts (xy 131.445 97.155) (xy 136.525 97.155))
     (stroke (width 0) (type default))
   )
-  (text "Power from SWI3-5-N-P5" (at 85.725 79.375 0)
+  (text "Power from SWI3-5-N-P5" (at 100.965 89.535 0)
     (effects (font (size 1.27 1.27)) (justify left bottom) (href "https://www.digikey.com/en/products/detail/cui-inc/SWI3-5-N-P5/7784528"))
   )
-  (text "Center + \nJack size 5" (at 90.805 97.79 0)
+  (text "Center + \nJack size 5" (at 106.045 107.95 0)
     (effects (font (size 1.27 1.27)) (justify left bottom))
   )
-  (symbol (lib_id "power:GND") (at 130.81 98.425 0) (unit 1)
+  (hierarchical_label "2V" (shape input) (at 136.525 97.155 0) (fields_autoplaced)
+    (effects (font (size 1.27 1.27)) (justify left))
+  )
+  (symbol (lib_id "power:GND") (at 131.445 108.585 0) (unit 1)
     (in_bom yes) (on_board yes) (dnp no) (fields_autoplaced)
-    (property "Reference" "#PWR0113" (at 130.81 104.775 0)
+    (property "Reference" "#PWR0114" (at 131.445 114.935 0)
       (effects (font (size 1.27 1.27)) hide)
     )
-    (property "Value" "GND" (at 130.81 102.87 0)
+    (property "Value" "GND" (at 131.445 113.03 0)
       (effects (font (size 1.27 1.27)) hide)
     )
-    (property "Footprint" "" (at 130.81 98.425 0)
+    (property "Footprint" "" (at 131.445 108.585 0)
       (effects (font (size 1.27 1.27)) hide)
     )
-    (property "Datasheet" "" (at 130.81 98.425 0)
+    (property "Datasheet" "" (at 131.445 108.585 0)
       (effects (font (size 1.27 1.27)) hide)
     )
@@
       (project "VMC1"
         (path "/030598bf-3d55-483a-af42-40ff6f2e377a/5124e20e-a7f5-40d6-8600-d692d8212b50"
-          (reference "#PWR0113") (unit 1)
+          (reference "#PWR0114") (unit 1)
         )
       )
     )
   )
-  (symbol (lib_id "Connector:Jack-DC") (at 95.25 89.535 0) (unit 1)
+  (symbol (lib_id "Connector:Jack-DC") (at 110.49 99.695 0) (unit 1)
     (in_bom yes) (on_board yes) (dnp no) (fields_autoplaced)
-    (property "Reference" "J?" (at 95.25 81.28 0)
+    (property "Reference" "J?" (at 110.49 91.44 0)
       (effects (font (size 1.27 1.27)))
     )
-    (property "Value" "5V" (at 95.25 83.82 0)
+    (property "Value" "5V" (at 110.49 93.98 0)
       (effects (font (size 1.27 1.27)))
     )
-    (property "Footprint" "" (at 96.52 90.551 0)
+    (property "Footprint" "" (at 111.76 100.711 0)
       (effects (font (size 1.27 1.27)) hide)
     )
-    (property "Datasheet" "~" (at 96.52 90.551 0)
+    (property "Datasheet" "~" (at 111.76 100.711 0)
       (effects (font (size 1.27 1.27)) hide)
     )
@@
     )
   )
-  (symbol (lib_id "Regulator_Linear:NCP1117-1.5_SOT223") (at 130.81 86.995 0) (unit 1)
-    (in_bom yes) (on_board yes) (dnp no)
-    (property "Reference" "U?" (at 130.81 83.82 0)
-      (effects (font (size 1.27 1.27)))
+  (symbol (lib_id "Device:C_Polarized") (at 131.445 103.505 0) (unit 1)
+    (in_bom yes) (on_board yes) (dnp no) (fields_autoplaced)
+    (property "Reference" "C?" (at 135.255 101.346 0)
+      (effects (font (size 1.27 1.27)) (justify left))
     )
-    (property "Value" "NCP1117ST20T3G" (at 140.335 93.345 0)
-      (effects (font (size 1.27 1.27)))
+    (property "Value" "10uF" (at 135.255 103.886 0)
+      (effects (font (size 1.27 1.27)) (justify left))
     )
-    (property "Footprint" "Package_TO_SOT_SMD:SOT-223-3_TabPin2" (at 130.81 81.915 0)
+    (property "Footprint" "" (at 132.4102 107.315 0)
       (effects (font (size 1.27 1.27)) hide)
     )
-    (property "Datasheet" "http://www.onsemi.com/pub_link/Collateral/NCP1117-D.PDF" (at 133.35 93.345 0)
+    (property "Datasheet" "~" (at 131.445 103.505 0)
       (effects (font (size 1.27 1.27)) hide)
     )
     (pin "1")
     (pin "2")
-    (pin "3")
     (instances
       (project "VMC1"
         (path "/030598bf-3d55-483a-af42-40ff6f2e377a/5124e20e-a7f5-40d6-8600-d692d8212b50"
-          (reference "U?") (unit 1)
+          (reference "C?") (unit 1)
         )
       )
+    )
+  )
+  (symbol (lib_id "power:GND") (at 119.38 108.585 0) (unit 1)
+    (in_bom yes) (on_board yes) (dnp no) (fields_autoplaced)
+    (property "Reference" "#PWR0115" (at 119.38 114.935 0)
+      (effects (font (size 1.27 1.27)) hide)
+    )
+    (property "Value" "GND" (at 119.38 113.03 0)
+      (effects (font (size 1.27 1.27)) hide)
+    )
+    (property "Footprint" "" (at 119.38 108.585 0)
+      (effects (font (size 1.27 1.27)) hide)
+    )
+    (property "Datasheet" "" (at 119.38 108.585 0)
+      (effects (font (size 1.27 1.27)) hide)
+    )
+    (pin "1")
+    (instances
+      (project "VMC1"
+        (path "/030598bf-3d55-483a-af42-40ff6f2e377a/5124e20e-a7f5-40d6-8600-d692d8212b50"
+          (reference "#PWR0115") (unit 1)
+        )
+      )
