File: VMC1.kicad_sch (KiCad schematic)
At the start: 0 parts

Commit message: V0.1
really jjust updating a bunch of stuff
Other:
- removed sheet LedPower
- sheet switches ports: added TLC5940 Bus; removed none
- title: (none) -> VMC-1

Commit message: First Round ERC Checks
Other:
- sheet switches ports: added none; removed TLC5940 Bus
Changed lines of the file:
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@@
-      (effects (font (size 1.27 1.27)) (justify right))
-    )
-    (pin "TLC5940 Bus" input (at 98.425 85.725 0)
       (effects (font (size 1.27 1.27)) (justify right))
     )
