File: pots 3.kicad_sch (KiCad schematic)
At the start: 17 parts

Commit message: V0.1
really jjust updating a bunch of stuff
Other:
- title: (none) -> VMC-1
Changed lines of the file:
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@@
 (kicad_sch (version 20230121) (generator eeschema)
   (paper "USLetter")
+  (title_block
+    (title "VMC-1")
+    (date "2023-12-03")
+  )
   (no_connect (at 137.16 83.82))
   (wire (pts (xy 119.38 78.74) (xy 96.52 78.74))

Commit message: Post Kicad Community Telling Me Shit is Wrong
way more stuff needs love, DECOUPERS DUMA88s
Parts:
- removed U?: CD74HC4067M, Package_SO:SOIC-24W_7.5x15.4mm_P1.27mm, symbol 74xx:CD74HC4067M
Connections:
- no-connect marks 1 -> 0
Other:
- note added: "ADC MUX you can get I2C/ SPI ADC which have many channels, you might want to go that route for your pots"
Changed lines of the file:
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@@
     (date "2023-12-03")
   )
-  (no_connect (at 137.16 83.82))
-  (wire (pts (xy 119.38 78.74) (xy 96.52 78.74))
-    (stroke (width 0) (type default))
-  )
   (wire (pts (xy 82.55 116.84) (xy 82.55 137.16))
     (stroke (width 0) (type default))
@@
     (stroke (width 0) (type default))
   )
-  (wire (pts (xy 119.38 83.82) (xy 119.38 78.74))
-    (stroke (width 0) (type default))
-  )
   (wire (pts (xy 127 137.16) (xy 127 125.73))
     (stroke (width 0) (type default))
@@
     (stroke (width 0) (type default))
   )
-  (wire (pts (xy 152.4 96.52) (xy 149.86 96.52))
-    (stroke (width 0) (type default))
-  )
-  (wire (pts (xy 121.92 76.2) (xy 121.92 83.82))
-    (stroke (width 0) (type default))
-  )
   (wire (pts (xy 127 120.65) (xy 127 109.22))
     (stroke (width 0) (type default))
@@
     (stroke (width 0) (type default))
   )
-  (wire (pts (xy 96.52 73.66) (xy 124.46 73.66))
-    (stroke (width 0) (type default))
-  )
-  (wire (pts (xy 93.98 96.52) (xy 96.52 96.52))
-    (stroke (width 0) (type default))
-  )
   (wire (pts (xy 143.51 123.19) (xy 143.51 137.16))
     (stroke (width 0) (type default))
@@
     (stroke (width 0) (type default))
   )
-  (wire (pts (xy 152.4 96.52) (xy 152.4 97.79))
-    (stroke (width 0) (type default))
-  )
   (wire (pts (xy 161.29 120.65) (xy 161.29 137.16))
     (stroke (width 0) (type default))
@@
     (stroke (width 0) (type default))
   )
-  (wire (pts (xy 96.52 76.2) (xy 121.92 76.2))
-    (stroke (width 0) (type default))
-  )
   (wire (pts (xy 143.51 123.19) (xy 121.92 123.19))
     (stroke (width 0) (type default))
@@
     (stroke (width 0) (type default))
   )
-  (wire (pts (xy 127 83.82) (xy 127 71.12))
-    (stroke (width 0) (type default))
-  )
   (wire (pts (xy 124.46 121.92) (xy 152.4 121.92))
     (stroke (width 0) (type default))
@@
     (stroke (width 0) (type default))
   )
-  (wire (pts (xy 124.46 73.66) (xy 124.46 83.82))
-    (stroke (width 0) (type default))
-  )
-  (wire (pts (xy 109.22 68.58) (xy 109.22 83.82))
-    (stroke (width 0) (type default))
-  )
   (wire (pts (xy 118.11 127) (xy 113.03 127))
     (stroke (width 0) (type default))
@@
     (stroke (width 0) (type default))
   )
-  (wire (pts (xy 127 71.12) (xy 96.52 71.12))
-    (stroke (width 0) (type default))
-  )
   (wire (pts (xy 119.38 124.46) (xy 135.89 124.46))
     (stroke (width 0) (type default))
@@
     (stroke (width 0) (type default))
   )
-  (label "S0" (at 101.6 78.74 0) (fields_autoplaced)
+  (text "ADC MUX\n\nyou can get I2C/ SPI ADC which have many channels, you might want to go that route for your pots\n"
+    (at 100.965 99.06 0)
     (effects (font (size 1.27 1.27)) (justify left bottom))
-  )
-  (label "S2" (at 101.6 73.66 0) (fields_autoplaced)
-    (effects (font (size 1.27 1.27)) (justify left bottom))
-  )
-  (label "S1" (at 101.6 76.2 0) (fields_autoplaced)
-    (effects (font (size 1.27 1.27)) (justify left bottom))
-  )
-  (label "S3" (at 101.6 71.12 0) (fields_autoplaced)
-    (effects (font (size 1.27 1.27)) (justify left bottom))
-  )
-  (hierarchical_label "S3" (shape input) (at 96.52 71.12 180) (fields_autoplaced)
-    (effects (font (size 1.27 1.27)) (justify right))
-  )
-  (hierarchical_label "S2" (shape input) (at 96.52 73.66 180) (fields_autoplaced)
-    (effects (font (size 1.27 1.27)) (justify right))
-  )
-  (hierarchical_label "S1" (shape input) (at 96.52 76.2 180) (fields_autoplaced)
-    (effects (font (size 1.27 1.27)) (justify right))
-  )
-  (hierarchical_label "S0" (shape input) (at 96.52 78.74 180) (fields_autoplaced)
-    (effects (font (size 1.27 1.27)) (justify right))
-  )
-  (hierarchical_label "Pots 3 COM" (shape input) (at 109.22 68.58 90) (fields_autoplaced)
-    (effects (font (size 1.27 1.27)) (justify left))
   )
   (symbol (lib_id "power:+3.3V") (at 130.81 133.35 0) (unit 1)
@@
     )
   )
-  (symbol (lib_id "74xx:CD74HC4067M") (at 121.92 96.52 90) (mirror x) (unit 1)
-    (in_bom yes) (on_board yes) (dnp no)
-    (property "Reference" "U?" (at 121.92 96.52 90)
-      (effects (font (size 1.27 1.27)))
-    )
-    (property "Value" "CD74HC4067M" (at 151.13 106.68 90)
-      (effects (font (size 1.27 1.27)))
-    )
-    (property "Footprint" "Package_SO:SOIC-24W_7.5x15.4mm_P1.27mm" (at 147.32 119.38 0)
-      (effects (font (size 1.27 1.27) italic) hide)
-    )
-    (property "Datasheet" "http://www.ti.com/lit/ds/symlink/cd74hc4067.pdf" (at 100.33 87.63 0)
-      (effects (font (size 1.27 1.27)) hide)
-    )
-    (pin "1")
-    (pin "10")
-    (pin "11")
-    (pin "12")
-    (pin "13")
-    (pin "14")
-    (pin "15")
-    (pin "16")
-    (pin "17")
-    (pin "18")
-    (pin "19")
-    (pin "2")
-    (pin "20")
-    (pin "21")
-    (pin "22")
-    (pin "23")
-    (pin "24")
-    (pin "3")
-    (pin "4")
-    (pin "5")
-    (pin "6")
-    (pin "7")
-    (pin "8")
-    (pin "9")
-    (instances
-      (project "VMC1"
-        (path "/030598bf-3d55-483a-af42-40ff6f2e377a/0e4dff31-92f3-4306-89d1-37404e655862"
-          (reference "U?") (unit 1)
-        )
-        (path "/030598bf-3d55-483a-af42-40ff6f2e377a/35d099d8-fbd8-4467-b743-48425c2f6fdb"
-          (reference "U4") (unit 1)
-        )
-      )
-      (project "V"
-        (path "/f9418f3a-fa41-4a3d-8541-c10ffd215f7d"
-          (reference "U?") (unit 1)
-        )
-        (path "/f9418f3a-fa41-4a3d-8541-c10ffd215f7d/7ffcc307-6cac-4824-b607-a8f1674c733d"
-          (reference "U?") (unit 1)
-        )
-      )
-    )
-  )
   (symbol (lib_id "power:GND") (at 182.88 140.97 0) (unit 1)
     (in_bom yes) (on_board yes) (dnp no) (fields_autoplaced)
@@
     )
   )
-  (symbol (lib_id "power:+3.3V") (at 93.98 96.52 0) (unit 1)
-    (in_bom yes) (on_board yes) (dnp no)
-    (property "Reference" "#PWR042" (at 93.98 100.33 0)
-      (effects (font (size 1.27 1.27)) hide)
-    )
-    (property "Value" "+3.3V" (at 93.98 92.71 0)
-      (effects (font (size 1.27 1.27)))
-    )
-    (property "Footprint" "" (at 93.98 96.52 0)
-      (effects (font (size 1.27 1.27)) hide)
-    )
-    (property "Datasheet" "" (at 93.98 96.52 0)
-      (effects (font (size 1.27 1.27)) hide)
-    )
-    (pin "1")
-    (instances
-      (project "VMC1"
-        (path "/030598bf-3d55-483a-af42-40ff6f2e377a/0e4dff31-92f3-4306-89d1-37404e655862"
-          (reference "#PWR042") (unit 1)
-        )
-        (path "/030598bf-3d55-483a-af42-40ff6f2e377a/35d099d8-fbd8-4467-b743-48425c2f6fdb"
-          (reference "#PWR076") (unit 1)
-        )
-      )
-      (project "V"
-        (path "/f9418f3a-fa41-4a3d-8541-c10ffd215f7d/7ffcc307-6cac-4824-b607-a8f1674c733d"
-          (reference "#PWR05") (unit 1)
-        )
-      )
-    )
-  )
   (symbol (lib_id "power:GND") (at 208.28 140.97 0) (unit 1)
     (in_bom yes) (on_board yes) (dnp no) (fields_autoplaced)
@@
         )
       )
-    )
-  )
-  (symbol (lib_id "power:GND") (at 152.4 97.79 0) (unit 1)
-    (in_bom yes) (on_board yes) (dnp no) (fields_autoplaced)
-    (property "Reference" "#PWR043" (at 152.4 104.14 0)
-      (effects (font (size 1.27 1.27)) hide)
-    )
-    (property "Value" "GND" (at 152.4 102.87 0)
-      (effects (font (size 1.27 1.27)) hide)
-    )
-    (property "Footprint" "" (at 152.4 97.79 0)
-      (effects (font (size 1.27 1.27)) hide)
-    )
-    (property "Datasheet" "" (at 152.4 97.79 0)
-      (effects (font (size 1.27 1.27)) hide)
-    )
-    (pin "1")
-    (instances
-      (project "VMC1"
-        (path "/030598bf-3d55-483a-af42-40ff6f2e377a/0e4dff31-92f3-4306-89d1-37404e655862"
-          (reference "#PWR043") (unit 1)
-        )
-        (path "/030598bf-3d55-483a-af42-40ff6f2e377a/35d099d8-fbd8-4467-b743-48425c2f6fdb"
-          (reference "#PWR077") (unit 1)
-        )
-      )
-      (project "V"
-        (path "/f9418f3a-fa41-4a3d-8541-c10ffd215f7d/7ffcc307-6cac-4824-b607-a8f1674c733d"
-          (reference "#PWR06") (unit 1)
-        )
-      )
