File: pots.kicad_sch (KiCad schematic)
At the start: 17 parts

Commit message: V0.1
really jjust updating a bunch of stuff
Other:
- title: (none) -> VMC-1
Changed lines of the file:
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@@
 (kicad_sch (version 20230121) (generator eeschema)
   (paper "USLetter")
+  (title_block
+    (title "VMC-1")
+    (date "2023-12-03")
+  )
   (no_connect (at 127 78.74))
   (wire (pts (xy 109.22 119.38) (xy 125.73 119.38))

Commit message: First Round ERC Checks
Parts:
- gave numbers to parts that had none: 17
Changed lines of the file:
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@@
   (symbol (lib_id "Device:R_Potentiometer") (at 111.76 132.08 180) (unit 1)
     (in_bom yes) (on_board yes) (dnp no)
-    (property "Reference" "RV?" (at 107.95 135.89 0)
+    (property "Reference" "RV5" (at 107.95 135.89 0)
       (effects (font (size 1.27 1.27)))
     )
@@
       (project "VMC1"
         (path "/030598bf-3d55-483a-af42-40ff6f2e377a/dcebf1f0-1fde-4bf1-a09a-c049aef368a5"
-          (reference "RV?") (unit 1)
+          (reference "RV5") (unit 1)
         )
       )
@@
   (symbol (lib_id "Device:R_Potentiometer") (at 172.72 132.08 180) (unit 1)
     (in_bom yes) (on_board yes) (dnp no)
-    (property "Reference" "RV?" (at 168.91 135.89 0)
+    (property "Reference" "RV12" (at 168.91 135.89 0)
       (effects (font (size 1.27 1.27)))
     )
@@
       (project "VMC1"
         (path "/030598bf-3d55-483a-af42-40ff6f2e377a/dcebf1f0-1fde-4bf1-a09a-c049aef368a5"
-          (reference "RV?") (unit 1)
+          (reference "RV12") (unit 1)
         )
       )
@@
   (symbol (lib_id "Device:R_Potentiometer") (at 102.87 132.08 180) (unit 1)
     (in_bom yes) (on_board yes) (dnp no)
-    (property "Reference" "RV?" (at 99.06 135.89 0)
+    (property "Reference" "RV4" (at 99.06 135.89 0)
       (effects (font (size 1.27 1.27)))
     )
@@
       (project "VMC1"
         (path "/030598bf-3d55-483a-af42-40ff6f2e377a/dcebf1f0-1fde-4bf1-a09a-c049aef368a5"
-          (reference "RV?") (unit 1)
+          (reference "RV4") (unit 1)
         )
       )
@@
   (symbol (lib_id "Device:R_Potentiometer") (at 189.23 132.08 180) (unit 1)
     (in_bom yes) (on_board yes) (dnp no)
-    (property "Reference" "RV?" (at 185.42 135.89 0)
+    (property "Reference" "RV14" (at 185.42 135.89 0)
       (effects (font (size 1.27 1.27)))
     )
@@
       (project "VMC1"
         (path "/030598bf-3d55-483a-af42-40ff6f2e377a/dcebf1f0-1fde-4bf1-a09a-c049aef368a5"
-          (reference "RV?") (unit 1)
+          (reference "RV14") (unit 1)
         )
       )
@@
   (symbol (lib_id "Device:R_Potentiometer") (at 137.16 132.08 180) (unit 1)
     (in_bom yes) (on_board yes) (dnp no)
-    (property "Reference" "RV?" (at 133.35 135.89 0)
+    (property "Reference" "RV8" (at 133.35 135.89 0)
       (effects (font (size 1.27 1.27)))
     )
@@
       (project "VMC1"
         (path "/030598bf-3d55-483a-af42-40ff6f2e377a/dcebf1f0-1fde-4bf1-a09a-c049aef368a5"
-          (reference "RV?") (unit 1)
+          (reference "RV8") (unit 1)
         )
       )
@@
   (symbol (lib_id "Device:R_Potentiometer") (at 129.54 132.08 180) (unit 1)
     (in_bom yes) (on_board yes) (dnp no)
-    (property "Reference" "RV?" (at 125.73 135.89 0)
+    (property "Reference" "RV7" (at 125.73 135.89 0)
       (effects (font (size 1.27 1.27)))
     )
@@
       (project "VMC1"
         (path "/030598bf-3d55-483a-af42-40ff6f2e377a/dcebf1f0-1fde-4bf1-a09a-c049aef368a5"
-          (reference "RV?") (unit 1)
+          (reference "RV7") (unit 1)
         )
       )
@@
   (symbol (lib_id "Device:R_Potentiometer") (at 85.09 132.08 180) (unit 1)
     (in_bom yes) (on_board yes) (dnp no)
-    (property "Reference" "RV?" (at 81.28 135.89 0)
+    (property "Reference" "RV2" (at 81.28 135.89 0)
       (effects (font (size 1.27 1.27)))
     )
@@
       (project "VMC1"
         (path "/030598bf-3d55-483a-af42-40ff6f2e377a/dcebf1f0-1fde-4bf1-a09a-c049aef368a5"
-          (reference "RV?") (unit 1)
+          (reference "RV2") (unit 1)
         )
       )
@@
   (symbol (lib_id "Device:R_Potentiometer") (at 181.61 132.08 180) (unit 1)
     (in_bom yes) (on_board yes) (dnp no)
-    (property "Reference" "RV?" (at 177.8 135.89 0)
+    (property "Reference" "RV13" (at 177.8 135.89 0)
       (effects (font (size 1.27 1.27)))
     )
@@
       (project "VMC1"
         (path "/030598bf-3d55-483a-af42-40ff6f2e377a/dcebf1f0-1fde-4bf1-a09a-c049aef368a5"
-          (reference "RV?") (unit 1)
+          (reference "RV13") (unit 1)
         )
       )
@@
   (symbol (lib_id "Device:R_Potentiometer") (at 207.01 132.08 180) (unit 1)
     (in_bom yes) (on_board yes) (dnp no)
-    (property "Reference" "RV?" (at 203.2 135.89 0)
+    (property "Reference" "RV16" (at 203.2 135.89 0)
       (effects (font (size 1.27 1.27)))
     )
@@
       (project "VMC1"
         (path "/030598bf-3d55-483a-af42-40ff6f2e377a/dcebf1f0-1fde-4bf1-a09a-c049aef368a5"
-          (reference "RV?") (unit 1)
+          (reference "RV16") (unit 1)
         )
       )
@@
   (symbol (lib_id "Device:R_Potentiometer") (at 93.98 132.08 180) (unit 1)
     (in_bom yes) (on_board yes) (dnp no)
-    (property "Reference" "RV?" (at 90.17 135.89 0)
+    (property "Reference" "RV3" (at 90.17 135.89 0)
       (effects (font (size 1.27 1.27)))
     )
@@
       (project "VMC1"
         (path "/030598bf-3d55-483a-af42-40ff6f2e377a/dcebf1f0-1fde-4bf1-a09a-c049aef368a5"
-          (reference "RV?") (unit 1)
+          (reference "RV3") (unit 1)
         )
       )
@@
   (symbol (lib_id "Device:R_Potentiometer") (at 120.65 132.08 180) (unit 1)
     (in_bom yes) (on_board yes) (dnp no)
-    (property "Reference" "RV?" (at 116.84 135.89 0)
+    (property "Reference" "RV6" (at 116.84 135.89 0)
       (effects (font (size 1.27 1.27)))
     )
@@
       (project "VMC1"
         (path "/030598bf-3d55-483a-af42-40ff6f2e377a/dcebf1f0-1fde-4bf1-a09a-c049aef368a5"
-          (reference "RV?") (unit 1)
+          (reference "RV6") (unit 1)
         )
       )
@@
   (symbol (lib_id "Device:R_Potentiometer") (at 198.12 132.08 180) (unit 1)
     (in_bom yes) (on_board yes) (dnp no)
-    (property "Reference" "RV?" (at 194.31 135.89 0)
+    (property "Reference" "RV15" (at 194.31 135.89 0)
       (effects (font (size 1.27 1.27)))
     )
@@
       (project "VMC1"
         (path "/030598bf-3d55-483a-af42-40ff6f2e377a/dcebf1f0-1fde-4bf1-a09a-c049aef368a5"
-          (reference "RV?") (unit 1)
+          (reference "RV15") (unit 1)
         )
       )
@@
   (symbol (lib_id "Device:R_Potentiometer") (at 154.94 132.08 180) (unit 1)
     (in_bom yes) (on_board yes) (dnp no)
-    (property "Reference" "RV?" (at 151.13 135.89 0)
+    (property "Reference" "RV10" (at 151.13 135.89 0)
       (effects (font (size 1.27 1.27)))
     )
@@
       (project "VMC1"
         (path "/030598bf-3d55-483a-af42-40ff6f2e377a/dcebf1f0-1fde-4bf1-a09a-c049aef368a5"
-          (reference "RV?") (unit 1)
+          (reference "RV10") (unit 1)
         )
       )
@@
   (symbol (lib_id "Device:R_Potentiometer") (at 163.83 132.08 180) (unit 1)
     (in_bom yes) (on_board yes) (dnp no)
-    (property "Reference" "RV?" (at 160.02 135.89 0)
+    (property "Reference" "RV11" (at 160.02 135.89 0)
       (effects (font (size 1.27 1.27)))
     )
@@
       (project "VMC1"
         (path "/030598bf-3d55-483a-af42-40ff6f2e377a/dcebf1f0-1fde-4bf1-a09a-c049aef368a5"
-          (reference "RV?") (unit 1)
+          (reference "RV11") (unit 1)
         )
       )
@@
   (symbol (lib_id "Device:R_Potentiometer") (at 146.05 132.08 180) (unit 1)
     (in_bom yes) (on_board yes) (dnp no)
-    (property "Reference" "RV?" (at 142.24 135.89 0)
+    (property "Reference" "RV9" (at 142.24 135.89 0)
       (effects (font (size 1.27 1.27)))
     )
@@
       (project "VMC1"
         (path "/030598bf-3d55-483a-af42-40ff6f2e377a/dcebf1f0-1fde-4bf1-a09a-c049aef368a5"
-          (reference "RV?") (unit 1)
+          (reference "RV9") (unit 1)
         )
       )
@@
   (symbol (lib_id "Device:R_Potentiometer") (at 76.2 132.08 180) (unit 1)
     (in_bom yes) (on_board yes) (dnp no)
-    (property "Reference" "RV?" (at 72.39 135.89 0)
+    (property "Reference" "RV1" (at 72.39 135.89 0)
       (effects (font (size 1.27 1.27)))
     )
@@
       (project "VMC1"
         (path "/030598bf-3d55-483a-af42-40ff6f2e377a/dcebf1f0-1fde-4bf1-a09a-c049aef368a5"
-          (reference "RV?") (unit 1)
+          (reference "RV1") (unit 1)
         )
       )
@@
   (symbol (lib_id "74xx:CD74HC4067M") (at 111.76 91.44 90) (mirror x) (unit 1)
     (in_bom yes) (on_board yes) (dnp no)
-    (property "Reference" "U?" (at 111.76 91.44 90)
+    (property "Reference" "U2" (at 111.76 91.44 90)
       (effects (font (size 1.27 1.27)))
     )
@@
       (project "VMC1"
         (path "/030598bf-3d55-483a-af42-40ff6f2e377a/dcebf1f0-1fde-4bf1-a09a-c049aef368a5"
-          (reference "U?") (unit 1)
-        )
-      )
+          (reference "U2") (unit 1)
+        )
+      )

Commit message: Post Kicad Community Telling Me Shit is Wrong
way more stuff needs love, DECOUPERS DUMA88s
Parts:
- removed RV1, RV10, RV11, RV12, RV13, RV14, RV15, RV16, RV2, RV3, RV4, RV5, RV6, RV7, RV8, RV9: ~, Potentiometer_THT:Potentiometer_Bourns_PTA3043_Single_Slide, symbol Device:R_Potentiometer
- removed U2: CD74HC4067M, Package_SO:SOIC-24W_7.5x15.4mm_P1.27mm, symbol 74xx:CD74HC4067M
Connections:
- no-connect marks 1 -> 0
