File: pots2.kicad_sch (KiCad schematic)
At the start: 17 parts

Commit message: V0.1
really jjust updating a bunch of stuff
Other:
- title: (none) -> VMC-1
Changed lines of the file:
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@@
 (kicad_sch (version 20230121) (generator eeschema)
   (paper "USLetter")
+  (title_block
+    (title "VMC-1")
+    (date "2023-12-03")
+  )
   (no_connect (at 128.905 85.09))
   (wire (pts (xy 99.695 120.65) (xy 92.075 120.65))

Commit message: First Round ERC Checks
Parts:
- gave numbers to parts that had none: 17

Commit message: Post Kicad Community Telling Me Shit is Wrong
way more stuff needs love, DECOUPERS DUMA88s
Parts:
- removed RV17, RV18, RV19, RV20, RV21, RV22, RV23, RV24, RV25, RV26, RV27, RV28, RV29, RV30, RV31, RV32: ~, Potentiometer_THT:Potentiometer_Bourns_PTA3043_Single_Slide, symbol Device:R_Potentiometer
- removed U3: CD74HC4067M, Package_SO:SOIC-24W_7.5x15.4mm_P1.27mm, symbol 74xx:CD74HC4067M
Connections:
- no-connect marks 1 -> 0
